File: Hardware/AetherIO/Power.kicad_sch (KiCad schematic)
At the start: 0 parts

Commit message: start RF_Switch
Parts:
- added C10, C15, C19, C22, C25, C30: 1uF, persional_library:C0603, symbol persional_library:C0603
- added C11, C26: 100nF, persional_library:C0603, symbol persional_library:C0603
- added C12, C13, C14, C17, C18, C20, C21, C23, C24, C27, C28, C29, C8, C9: 22uF, persional_library:C0603, symbol persional_library:C0603
- added C16, C31: 220pF, persional_library:C0603, symbol persional_library:C0603
- added CN2: ~, persional_library:CONN-TH_2P-P2.50_HX25003-2A, symbol persional_library:Connect_ZX-XH2.54-2P
- added DC1: ~, persional_library:DC-005_2.5, symbol persional_library:Connect_DC-005_2.5
- added L1, L2: 3.3uH, persional_library:IND-SMD_L7.0-W6.6, symbol persional_library:L0630-3.3UH
- added R38, R42: 10Ω, persional_library:R0603, symbol persional_library:R0603
- added R39, R43: 100kΩ, persional_library:R0603, symbol persional_library:R0603
- added R40: 22.1kΩ, persional_library:R0603, symbol persional_library:R0603
- added R41, R45: 10kΩ, persional_library:R0603, symbol persional_library:R0603
- added R44: 13.7kΩ, persional_library:R0603, symbol persional_library:R0603
- added SW8: ~, persional_library:SW-TH_SK12D07VG4, symbol persional_library:Switch_SPDT_SK12D07VG4
- added U4, U5: ~, persional_library:SOT-23-8_L2.9-W1.6-P0.65-LS2.8-BR, symbol persional_library:DCDC_MP2236GJ-Z
- added U6: ~, persional_library:SOT-23-5_L2.9-W1.6-P0.95-LS2.8-BR, symbol persional_library:DCDC_TPS7A2033PDBVR
Connections:
- new net: C15.1, U4.7 (VCC)
- new net: R45.1, U5.6 (EN)
- new net: R41.1, U4.6 (EN)
- new net: C11.1, L1.1, U4.3 (SW)
- new net: C11.2, R38.1
- new net: C31.2, R43.1, R44.2, U5.8 (FB)
- new net: C26.1, L2.1, U5.3 (SW)
- new net: C26.2, R42.1
- new net: C30.1, U5.7 (VCC)
- new net: C16.2, R39.1, R40.2, U4.8 (FB)
- new net: R38.2, U4.5 (BST)
- new net: R42.2, U5.5 (BST)
- new net +5V: C17.1, C18.1, C19.1, C27.1, C28.1, C29.1, C31.1, L2.2, R43.2, U6.1 (IN), U6.3 (EN)
- new net 3V3: C12.1, C13.1, C14.1, C16.1, C20.1, C21.1, C22.1, L1.2, R39.2, U6.5 (OUT)
- new net GND: C10.2, C12.2, C13.2, C14.2, C15.2, C17.2, C18.2, C19.2, C20.2, C21.2, C22.2, C23.2, C24.2, C25.2, C27.2, C28.2, C29.2, C30.2, C8.2, C9.2, CN2.1, DC1.2, DC1.3, R40.1, R44.1, U4.1 (AGND), U4.4 (GND), U5.1 (AGND), U5.4 (GND), U6.2 (GND)
- new net VCC: C10.1, C23.1, C24.1, C25.1, C8.1, C9.1, R41.2, R45.2, SW8.2, U4.2 (IN), U5.2 (IN)
- new net VIN: CN2.2, DC1.1 (4), SW8.3
- no-connect marks 0 -> 3
